File: 2024-2025/hardware/hardware.kicad_pcb (KiCad board)
At the start: 2 copper layers, 100 x 81.1 mm, 23 parts, among them J1 Conn_01x04, J2 Conn_01x05, J3 Conn_01x15, J4 Conn_01x15, Q1 BSS138, Q2 BSS138, U1 MPR121QR2, U2 AP2112K-3.3

Commit message: Forgot to commit this
Parts:
- J1: footprint Connector_PinSocket_2.54mm:PinSocket_1x04_P2.54mm_Vertical_SMD_Pin1Left -> Connector_PinSocket_2.54mm:PinSocket_1x04_P2.54mm_Vertical
- J2: footprint Connector_PinSocket_2.54mm:PinSocket_1x05_P2.54mm_Vertical_SMD_Pin1Right -> Connector_PinSocket_2.54mm:PinSocket_1x05_P2.54mm_Vertical
- J3, J4: footprint Connector_PinSocket_2.54mm:PinSocket_1x15_P2.54mm_Vertical_SMD_Pin1Left -> Connector_PinSocket_2.54mm:PinSocket_1x15_P2.54mm_Vertical
- moved J3 18.8 mm to (54.8, 76.9)
- moved J4 18.8 mm to (54.8, 89.6)
- moved J2 2.32 mm to (20.4, 51.4)
Routing:
- net SCL: track 17.0 -> 23.3 mm, vias 0 -> 2
- net ELE3: track 291.5 -> 285.6 mm, vias 3 -> 5
- net SDA: track 24.5 -> 30.1 mm
- net ELE1: track 53.8 -> 58.0 mm
- net ELE0: track 21.8 -> 18.8 mm
- net GND: track 67.0 -> 64.6 mm
- net ELE2: track 411.7 -> 412.7 mm
- net ELE4: track 194.5 -> 195.4 mm
